Commit message: Add robot_description package with concept URDF, sensors, arm placeholder, and RViz view

File: ros2_ws/src/robot_description/urdf/constants.xacro (robot description, xacro)
@@ -1,44 +1,45 @@
 <?xml version="1.0"?>
 <robot xmlns:xacro="http://www.ros.org/wiki/xacro">
-  <!-- chassis -->
-  <xacro:property name="chassis_length" value="0.70"/>
-  <xacro:property name="chassis_width"  value="0.45"/>
-  <xacro:property name="chassis_height" value="0.14"/>
-  <!-- wheels -->
-  <xacro:property name="wheel_radius" value="0.06"/>
-  <xacro:property name="wheel_width"  value="0.035"/>
-  <xacro:property name="wheel_x" value="0.26"/>
-  <xacro:property name="wheel_y" value="0.20"/>
-  <xacro:property name="wheel_z" value="-0.07"/>
-  <!-- bins -->
-  <xacro:property name="bin_length" value="0.22"/>
-  <xacro:property name="bin_width"  value="0.18"/>
-  <xacro:property name="bin_height" value="0.18"/>
+  <!-- Approximate dimensions (meters) -->
+  <xacro:property name="chassis_L" value="0.55"/>
+  <xacro:property name="chassis_W" value="0.45"/>
+  <xacro:property name="chassis_H" value="0.18"/>
+  <xacro:property name="wheel_R" value="0.10"/>
+  <xacro:property name="wheel_W" value="0.05"/>
+  <xacro:property name="wheel_mass" value="1.0"/>
+  <!-- LiDAR mount -->
+  <xacro:property name="lidar_x" value="0.20"/>
+  <xacro:property name="lidar_y" value="0.00"/>
+  <xacro:property name="lidar_z" value="0.22"/>
+  <xacro:property name="lidar_mass" value="0.25"/>
+  <!-- Camera mount -->
+  <xacro:property name="cam_x" value="0.18"/>
+  <xacro:property name="cam_y" value="0.00"/>
+  <xacro:property name="cam_z" value="0.26"/>
+  <xacro:property name="cam_mass" value="0.20"/>
+  <!-- Bins (rear left/right) -->
+  <xacro:property name="bin_L" value="0.22"/>
+  <xacro:property name="bin_W" value="0.16"/>
+  <xacro:property name="bin_H" value="0.20"/>
   <xacro:property name="bin_x" value="-0.18"/>
-  <xacro:property name="bin_y" value="0.11"/>
-  <xacro:property name="bin_z" value="0.13"/>
-  <!-- bin pedestals -->
-  <xacro:property name="bin_ped_radius" value="0.035"/>
-  <xacro:property name="bin_ped_height" value="0.10"/>
-  <xacro:property name="bin_ped_half" value="0.05"/>
-  <!-- lidar -->
-  <xacro:property name="lidar_x" value="0.10"/>
-  <xacro:property name="lidar_z" value="0.22"/>
-  <xacro:property name="lidar_ped_radius" value="0.02"/>
-  <xacro:property name="lidar_ped_height" value="0.10"/>
-  <xacro:property name="lidar_ped_half" value="0.05"/>
-  <!-- arm mount -->
-  <xacro:property name="arm_base_x" value="0.30"/>
-  <xacro:property name="arm_base_z" value="0.12"/>
-  <!-- arm dims -->
-  <xacro:property name="L1" value="0.10"/>
-  <xacro:property name="L2" value="0.18"/>
-  <xacro:property name="L3" value="0.16"/>
-  <xacro:property name="L4" value="0.08"/>
-  <xacro:property name="tool_len" value="0.10"/>
-  <xacro:property name="finger_len" value="0.08"/>
-  <xacro:property name="L2_half" value="0.09"/>
-  <xacro:property name="L3_half" value="0.08"/>
-  <xacro:property name="tool_half" value="0.05"/>
-  <xacro:property name="finger_half" value="0.04"/>
+  <xacro:property name="bin_z" value="0.20"/>
+  <xacro:property name="bin_left_y"  value="0.12"/>
+  <xacro:property name="bin_right_y" value="-0.12"/>
+  <xacro:property name="bin_mass" value="1.5"/>
+  <!-- Arm base -->
+  <xacro:property name="arm_x" value="0.12"/>
+  <xacro:property name="arm_y" value="0.00"/>
+  <xacro:property name="arm_z" value="0.22"/>
+  <xacro:property name="arm_base_height" value="0.08"/>
+  <xacro:property name="arm_link1_len" value="0.16"/>
+  <xacro:property name="arm_link2_len" value="0.16"/>
+  <xacro:property name="arm_link3_len" value="0.12"/>
+  <xacro:property name="arm_link4_len" value="0.08"/>
+  <xacro:property name="arm_link5_len" value="0.08"/>
+  <xacro:property name="arm_link6_len" value="0.06"/>
+  <xacro:property name="arm_link_mass" value="0.6"/>
+  <xacro:property name="gripper_mass" value="0.3"/>
+  <xacro:property name="finger_len" value="0.06"/>
+  <xacro:property name="finger_width" value="0.015"/>
+  <xacro:property name="finger_thickness" value="0.02"/>
 </robot>

File: ros2_ws/src/robot_description/urdf/green_guardian.urdf.xacro (robot description, xacro)
@@ -1,18 +1,11 @@
 <?xml version="1.0"?>
-<robot xmlns:xacro="http://www.ros.org/wiki/xacro" name="green_guardian">
+<robot name="green_guardian" xmlns:xacro="http://www.ros.org/wiki/xacro">
   <xacro:include filename="$(find robot_description)/urdf/constants.xacro"/>
   <xacro:include filename="$(find robot_description)/urdf/materials.xacro"/>
-  <xacro:include filename="$(find robot_description)/urdf/macros.xacro"/>
-  <xacro:include filename="$(find robot_description)/urdf/base_chassis.xacro"/>
-  <xacro:include filename="$(find robot_description)/urdf/wheels.xacro"/>
-  <xacro:include filename="$(find robot_description)/urdf/bins.xacro"/>
-  <xacro:include filename="$(find robot_description)/urdf/lidar.xacro"/>
-  <xacro:include filename="$(find robot_description)/urdf/gripper.xacro"/>
-  <xacro:include filename="$(find robot_description)/urdf/depth_camera.xacro"/>
-  <xacro:base_chassis/>
-  <xacro:wheels parent="base_link"/>
-  <xacro:bins parent="base_link"/>
-  <xacro:lidar parent="base_link"/>
-  <xacro:gripper parent="base_link"/>
-  <xacro:depth_camera parent="base_link"/>
+  <xacro:include filename="$(find robot_description)/urdf/chassis.xacro"/>
+  <xacro:include filename="$(find robot_description)/urdf/wheels/wheels.xacro"/>
+  <xacro:include filename="$(find robot_description)/urdf/bins/bins.xacro"/>
+  <xacro:include filename="$(find robot_description)/urdf/sensors/rplidar_a1.xacro"/>
+  <xacro:include filename="$(find robot_description)/urdf/sensors/depth_camera.xacro"/>
+  <xacro:include filename="$(find robot_description)/urdf/arm/arm_placeholder_6dof.xacro"/>
 </robot>

File: ros2_ws/src/robot_description/urdf/materials.xacro (robot description, xacro)
@@ -1,8 +1,8 @@
 <?xml version="1.0"?>
 <robot xmlns:xacro="http://www.ros.org/wiki/xacro">
-  <material name="black"><color rgba="0.05 0.05 0.05 1.0"/></material>
-  <material name="gray"><color rgba="0.6 0.6 0.6 1.0"/></material>
-  <material name="white"><color rgba="1 1 1 1"/></material>
-  <material name="green"><color rgba="0.0 0.8 0.0 1.0"/></material>
-  <material name="blue"><color rgba="0.1 0.3 0.9 1.0"/></material>
+  <material name="gg_green"><color rgba="0.10 0.70 0.25 1.0"/></material>
+  <material name="gg_gray"><color rgba="0.60 0.60 0.60 1.0"/></material>
+  <material name="gg_black"><color rgba="0.05 0.05 0.05 1.0"/></material>
+  <material name="gg_blue"><color rgba="0.10 0.30 0.80 1.0"/></material>
+  <material name="gg_orange"><color rgba="0.95 0.55 0.10 1.0"/></material>
 </robot>
