Commit message: edit bins height

File: ros2_ws/src/robot_description/urdf/sensors.xacro (robot description, xacro)
@@ -36,5 +36,5 @@
     <!-- standoff center Z = chassis_top (rel to base_link) + standoff_h/2 -->
     <!-- = 0.033 + 0.0725 = 0.1055 m above base_link -->
-  </joint>
+  </joint>c
   <!-- ───────────────────────────────────────────────────────────────
        LASER LINK (LiDAR body cylinder)

Commit message: fix sensor.xacro

File: ros2_ws/src/robot_description/urdf/sensors.xacro (robot description, xacro)
@@ -36,5 +36,5 @@
     <!-- standoff center Z = chassis_top (rel to base_link) + standoff_h/2 -->
     <!-- = 0.033 + 0.0725 = 0.1055 m above base_link -->
-  </joint>c
+  </joint>
   <!-- ───────────────────────────────────────────────────────────────
        LASER LINK (LiDAR body cylinder)

Commit message: update direction of lidar sensor

File: ros2_ws/src/robot_description/urdf/sensors.xacro (robot description, xacro)
@@ -67,5 +67,5 @@
     <parent link="lidar_standoff_link"/>
     <child  link="laser_link"/>
-    <origin xyz="0 0 ${lidar_z}" rpy="0 0 0"/>
+    <origin xyz="0 0 ${lidar_z}" rpy="0 0 3.14159"/>
     <!-- LiDAR center Z relative to standoff center -->
     <!-- = standoff_h/2 + lidar_h/2 = 0.0725 + 0.015 = 0.0875 m -->
