Commit message: added sim_control and ros2_control with odom fixed_frame

File: ros2_ws/src/robot_description/urdf/components/bins.xacro (robot description, xacro)
@@ -37,5 +37,4 @@
       <parent link="${parent}"/>
       <child link="left_bin_link"/>
-      <!-- Positioned near the rear, offset to the left -->
       <origin xyz="${bin_x} ${bin_y_offset} ${bin_z}" rpy="0 0 0"/>
     </joint>

File: ros2_ws/src/robot_description/urdf/config/dimensions.xacro (robot description, xacro)
@@ -6,13 +6,11 @@
   <xacro:property name="chassis_width"  value="0.4"/>
   <xacro:property name="chassis_height" value="0.12"/>
-  <!-- Height of base_link above ground (simple assumption for now) -->
-  <xacro:property name="base_link_z" value="${wheel_radius + chassis_height/2.0}"/>
   <!-- ===== Wheels (4 wheels, differential by left/right sides) ===== -->
   <xacro:property name="wheel_radius" value="0.065"/>
   <xacro:property name="wheel_width"  value="0.03"/>
   <!-- wheel positions relative to base_link origin -->
-  <xacro:property name="wheel_x_front" value="${chassis_length/2.0 - 0.06}"/>
-  <xacro:property name="wheel_x_rear"  value="${-chassis_length/2.0 + 0.06}"/>
-  <xacro:property name="wheel_y_left"  value="${chassis_width/2.0 + wheel_width/2.0}"/>
+  <xacro:property name="wheel_x_front" value="${chassis_length/2.0 - 0.08}"/>
+  <xacro:property name="wheel_x_rear"  value="${-chassis_length/2.0 + 0.08}"/>
+  <xacro:property name="wheel_y_left"  value="${chassis_width/2.0 + wheel_width/2.0 + 0.002}"/>
   <xacro:property name="wheel_y_right" value="${-wheel_y_left}"/>
   <xacro:property name="wheel_z" value="${-chassis_height/2.0}"/>
@@ -35,3 +33,5 @@
   <xacro:property name="depth_cam_y" value="0.00"/>
   <xacro:property name="depth_cam_z" value="${chassis_height/2.0 - 0.03/2.0}"/>
+  <!-- Height of base_link above ground (simple assumption for now) -->
+  <xacro:property name="base_link_z" value="${wheel_radius + chassis_height/2.0}"/>
 </robot>

File: ros2_ws/src/robot_description/urdf/robot.urdf.xacro (robot description, xacro)
@@ -1,4 +1,5 @@
 <?xml version="1.0"?>
 <robot name="green_guardian" xmlns:xacro="http://ros.org/wiki/xacro">
+  <xacro:include filename="$(find robot_description)/urdf/ros2_control/gz_ros2_control.xacro"/>
   <!-- =========================
        Config (shared variables)
@@ -12,5 +13,4 @@
   <xacro:include filename="$(find robot_description)/urdf/components/bins.xacro"/>
   <xacro:include filename="$(find robot_description)/urdf/components/wheels.xacro"/>
-  <xacro:include filename="$(find robot_description)/urdf/components/arm_gripper_placeholder.xacro"/>
   <!-- =========================
        Sensors
@@ -36,5 +36,4 @@
   <xacro:wheels parent="base_link"/>
   <!-- placeholder (we will implement later, can stay empty file for now) -->
-  <xacro:arm_gripper_placeholder parent="base_link"/>
   <xacro:lidar parent="base_link"/>
   <xacro:depth_camera parent="base_link"/>

File: ros2_ws/src/robot_description/urdf/sensors/depth_camera.xacro (robot description, xacro)
@@ -43,5 +43,11 @@
     </joint>
     <!-- Optional alias frame (sometimes drivers/users prefer 'camera_frame') -->
-    <link name="depth_camera_frame"/>
+    <link name="depth_camera_frame">
+      <inertial>
+        <origin xyz="0 0 0" rpy="0 0 0"/>
+        <mass value="0.0001"/>
+       <inertia ixx="1e-8" iyy="1e-8" izz="1e-8" ixy="0" ixz="0" iyz="0"/>
+      </inertial>
+    </link>
     <joint name="depth_camera_link_to_frame_joint" type="fixed">
       <parent link="depth_camera_link"/>
@@ -50,5 +56,11 @@
     </joint>
     <!-- Optical frame (REP-103): Z forward, X right, Y down -->
-    <link name="depth_camera_optical_frame"/>
+    <link name="depth_camera_optical_frame">
+      <inertial>
+        <origin xyz="0 0 0" rpy="0 0 0"/>
+        <mass value="0.0001"/>
+        <inertia ixx="1e-8" iyy="1e-8" izz="1e-8" ixy="0" ixz="0" iyz="0"/>
+      </inertial>
+    </link>
     <joint name="depth_camera_frame_to_optical_joint" type="fixed">
       <parent link="depth_camera_frame"/>

File: ros2_ws/src/robot_description/urdf/sensors/lidar.xacro (robot description, xacro)
@@ -48,5 +48,11 @@
     </joint>
     <!-- Optional alias frame often expected by LiDAR drivers -->
-    <link name="laser_frame"/>
+    <link name="laser_frame">
+      <inertial>
+        <origin xyz="0 0 0" rpy="0 0 0"/>
+        <mass value="0.0001"/>
+        <inertia ixx="1e-8" iyy="1e-8" izz="1e-8" ixy="0" ixz="0" iyz="0"/>
+      </inertial>
+    </link>
     <joint name="lidar_to_laser_frame_joint" type="fixed">
       <parent link="lidar_link"/>
