Commit message: add lidar and camera plugins to gazebo

File: ros2_ws/src/robot_description/urdf/config/dimensions.xacro (robot description, xacro)
@@ -20,8 +20,7 @@
   <xacro:property name="bin_height" value="0.15"/>
   <!-- bin mounting positions -->
-  <xacro:property name="bin_rear_margin" value="0.02"/>
-  <xacro:property name="bin_x" value="${-chassis_length/2.0 + bin_length/2.0 + bin_rear_margin}"/>
+  <xacro:property name="bin_x" value="${-chassis_length/2.0 - bin_length/2.0}"/>
   <xacro:property name="bin_y_offset" value="0.10"/>
-  <xacro:property name="bin_z" value="${chassis_height/2.0 + bin_height/2.0}"/>
+  <xacro:property name="bin_z" value="0.00"/>
   <!-- ===== LIDAR mount ===== -->
   <xacro:property name="lidar_x" value="-0.03"/>

File: ros2_ws/src/robot_description/urdf/ros2_control/gz_ros2_control.xacro (robot description, xacro)
@@ -35,4 +35,7 @@
       <parameters>$(arg controllers_yaml)</parameters>
     </plugin>
+    <!-- Publish ground-truth odometry from Gazebo so RViz matches collisions / contacts. -->
+    <plugin filename="gz-sim-odometry-publisher-system"
+            name="gz::sim::systems::OdometryPublisher"/>
   </gazebo>
 </robot>

File: ros2_ws/src/robot_description/urdf/sensors/depth_camera.xacro (robot description, xacro)
@@ -69,4 +69,28 @@
       <origin xyz="0 0 0" rpy="-1.5708 0 -1.5708"/>
     </joint>
+    <!-- Gazebo RGB camera (C920-like) -->
+    <gazebo reference="depth_camera_link">
+  <sensor type="camera" name="c920_rgb_camera">
+    <always_on>true</always_on>
+    <update_rate>30</update_rate>
+    <visualize>true</visualize>
+    <camera>
+      <horizontal_fov>1.396</horizontal_fov>
+      <image>
+        <width>640</width>
+        <height>480</height>
+        <format>R8G8B8</format>
+      </image>
+      <clip>
+        <near>0.1</near>
+        <far>50</far>
+      </clip>
+    </camera>
+  </sensor>
+</gazebo>
+<!-- Ensure the Sensors system is loaded -->
+<gazebo>
+  <plugin name="gz::sim::systems::Sensors" filename="libgz-sim-sensors-system.so"/>
+</gazebo>
   </xacro:macro>
 </robot>

File: ros2_ws/src/robot_description/urdf/sensors/lidar.xacro (robot description, xacro)
@@ -60,4 +60,36 @@
       <origin xyz="0 0 0" rpy="0 0 0"/>
     </joint>
+    <!-- Gazebo LiDAR sensor (publishes gz.msgs.LaserScan on /scan) -->
+    <gazebo reference="lidar_link">
+      <!-- Keep this link from being lumped away so the sensor has a stable frame -->
+      <disableFixedJointLumping>true</disableFixedJointLumping>
+      <sensor name="laser_frame" type="gpu_lidar">
+        <topic>scan</topic>
+        <update_rate>10</update_rate>
+        <ray>
+          <scan>
+            <horizontal>
+              <samples>720</samples>
+              <resolution>1</resolution>
+              <min_angle>-3.141592653589793</min_angle>
+              <max_angle>3.141592653589793</max_angle>
+            </horizontal>
+            <vertical>
+              <samples>1</samples>
+              <resolution>1</resolution>
+              <min_angle>0</min_angle>
+              <max_angle>0</max_angle>
+            </vertical>
+          </scan>
+          <range>
+            <min>0.08</min>
+            <max>10.0</max>
+            <resolution>0.01</resolution>
+          </range>
+        </ray>
+        <always_on>1</always_on>
+        <visualize>true</visualize>
+      </sensor>
+    </gazebo>
   </xacro:macro>
 </robot>
